Commit message: updated changes

File: urdf/rover_lidar.urdf (robot description, URDF)
Before this commit: robot rover_lidar, 8 links, 7 joints
Links:
- link base_link: geometry collision mesh filename=package://updated_robot_lidar/meshes/base_link.STL; visual mesh filename=package://updated_robot_lidar/meshes/base_link.STL
- link bottom_left_wheel: geometry collision mesh filename=package://updated_robot_lidar/meshes/bottom_left_wheel.STL; visual mesh filename=package://updated_robot_lidar/meshes/bottom_left_wheel.STL
- link bottom_right_wheel: geometry collision mesh filename=package://updated_robot_lidar/meshes/bottom_right_wheel.STL; visual mesh filename=package://updated_robot_lidar/meshes/bottom_right_wheel.STL
- link front_left_wheel: geometry collision mesh filename=package://updated_robot_lidar/meshes/front_left_wheel.STL; visual mesh filename=package://updated_robot_lidar/meshes/front_left_wheel.STL
- link front_right_wheel: geometry collision mesh filename=package://updated_robot_lidar/meshes/front_right_wheel.STL; visual mesh filename=package://updated_robot_lidar/meshes/front_right_wheel.STL
- link left_tread: geometry collision mesh filename=package://updated_robot_lidar/meshes/left_tread.STL; visual mesh filename=package://updated_robot_lidar/meshes/left_tread.STL
- link lidar_link: mass 0.094104181491117 -> 0.0941041819406961; geometry collision mesh filename=package://updated_robot_lidar/meshes/lidar_link.STL; visual mesh filename=package://updated_robot_lidar/meshes/lidar_link.STL
- link right_tread: geometry collision mesh filename=package://updated_robot_lidar/meshes/right_tread.STL; visual mesh filename=package://updated_robot_lidar/meshes/right_tread.STL
Joints:
- joint base_link_bottom_right_wheel: origin xyz=-0.113531519133702 -0.127 -0.029415678198117 rpy=1.5707963267949 0 0 -> xyz=-0.11353 -0.127 -0.029416 rpy=1.5708 0 0
- joint base_link_right_tread: origin xyz=0.00929378954049227 -0.1065 -0.000296284357995884 rpy=1.5707963267949 0 0 -> xyz=0.0092938 -0.1065 -0.00029628 rpy=1.5708 0 0
- joint base_link_to_bottom_left_wheel: origin xyz=-0.115435440029406 0.127 -0.023104093147408 rpy=1.5707963267949 0 3.14159265358979 -> xyz=-0.11544 0.127 -0.023104 rpy=1.5708 0 3.1416
- joint base_link_to_front_left_wheel: origin xyz=0.1188588681311 0.127 -0.019031967432299 rpy=1.5707963267949 0 3.14159265358979 -> xyz=0.11886 0.127 -0.019032 rpy=1.5708 0 3.1416
- joint base_link_to_front_right_wheel: origin xyz=0.117290515707591 -0.127 -0.025435192502925 rpy=1.5707963267949 -1.5707963267949 0 -> xyz=0.11729 -0.127 -0.025435 rpy=1.5708 -1.5708 0
- joint base_link_to_lidar_link: origin xyz=0.0011557 0 -0.008 rpy=0 0 3.1416 -> xyz=-0.044901 0.0003607 0.094632 rpy=0 0.048079 2.0209

Commit message: updated changes

File: urdf/rover_lidar.urdf (robot description, URDF)
Before this commit: robot updated_robot_lidar, 8 links, 7 joints
Links:
- removed link left_tread
- removed link lidar_link
- removed link right_tread
- link base_link: mass 0.84121706270277 -> 0.841217991440235; geometry collision mesh filename=file:///home/anonymous/project_ws/src/rover/meshes/meshes/b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; visual mesh filename=file:///home/anonymous/project_ws/src/rover/meshes/meshes/b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
- link bottom_left_wheel: geometry collision mesh filename=file:///home/anonymous/project_ws/src/rover/meshes/meshes/b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; visual mesh filename=file:///home/anonymous/project_ws/src/rover/meshes/meshes/b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
- link bottom_right_wheel: mass 0.0169810669319343 -> 0.0169810669319342; geometry collision mesh filename=file:///home/anonymous/project_ws/src/rover/meshes/meshes/b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; visual mesh filename=file:///home/anonymous/project_ws/src/rover/meshes/meshes/b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
- link front_left_wheel: geometry collision mesh filename=file:///home/anonymous/project_ws/src/rover/meshes/meshes/f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; visual mesh filename=file:///home/anonymous/project_ws/src/rover/meshes/meshes/f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
- link front_right_wheel: geometry collision mesh filename=file:///home/anonymous/project_ws/src/rover/meshes/meshes/f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; visual mesh filename=file:///home/anonymous/project_ws/src/rover/meshes/meshes/f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
Joints:
- removed joint base_link_bottom_right_wheel
- removed joint base_link_right_tread
- removed joint base_link_to_bottom_left_wheel
- removed joint base_link_to_left_tread
- removed joint base_link_to_lidar_link
- added joint base_link_to_bottom_right_wheel: type continuous, parent base_link, child bottom_left_wheel, origin xyz=-0.1177 0.127 -0.011032 rpy=1.5708 0 3.1416, axis 0 0 -1
- joint base_link_to_front_left_wheel: origin xyz=0.11886 0.127 -0.019032 rpy=1.5708 0 3.1416 -> xyz=0.11659 0.127 -0.015104 rpy=1.5708 0 3.1416
- joint base_link_to_front_right_wheel: origin xyz=0.11729 -0.127 -0.025435 rpy=1.5708 -1.5708 0 -> xyz=0.11659 -0.127 -0.015104 rpy=1.5708 0 0
